File: Supply.sch (KiCad schematic (older format))
At the start: 7 parts, among them P5 CONN_01X02, Q5 AO3401, U3 EPL3015, U4 TPS61222

Commit message: Update schematic and reroute print
 * Update opamp circuit for light sensor
 * Change opamp
 * Reroute everything

Signed-off-by: Philip Luyckx <philip.luyckx@gmail.com>
Parts:
- Q5: footprint SMD_Packages:SOT-323 -> CustomSmd:SOT23
Changed lines of the file:
@@
 $EndComp
 $Comp
-L +BATT #PWR35
+L +BATT #PWR035
 U 1 1 56631049
 P 1600 2050
-F 0 "#PWR35" H 1600 1900 50  0001 C CNN
+F 0 "#PWR035" H 1600 1900 50  0001 C CNN
 F 1 "+BATT" H 1600 2190 50  0000 C CNN
 F 2 "" H 1600 2050 60  0000 C CNN
@@
 $EndComp
 $Comp
-L GND #PWR36
+L GND #PWR036
 U 1 1 5663105F
 P 1600 2150
-F 0 "#PWR36" H 1600 1900 50  0001 C CNN
+F 0 "#PWR036" H 1600 1900 50  0001 C CNN
 F 1 "GND" H 1600 2000 50  0000 C CNN
 F 2 "" H 1600 2150 60  0000 C CNN
@@
 	1400 2400 1400 1800
 $Comp
-L +BATT #PWR34
+L +BATT #PWR037
 U 1 1 56635CFE
 P 1500 1000
-F 0 "#PWR34" H 1500 850 50  0001 C CNN
+F 0 "#PWR037" H 1500 850 50  0001 C CNN
 F 1 "+BATT" H 1500 1140 50  0000 C CNN
 F 2 "" H 1500 1000 60  0000 C CNN
@@
 $EndComp
 $Comp
-L GND #PWR33
+L GND #PWR038
 U 1 1 56635D42
 P 1100 1050
-F 0 "#PWR33" H 1100 800 50  0001 C CNN
+F 0 "#PWR038" H 1100 800 50  0001 C CNN
 F 1 "GND" H 1100 900 50  0000 C CNN
 F 2 "" H 1100 1050 60  0000 C CNN
@@
 $EndComp
 $Comp
-L PWR_FLAG #FLG1
+L PWR_FLAG #FLG039
 U 1 1 56635D80
 P 1100 1050
-F 0 "#FLG1" H 1100 1145 50  0001 C CNN
+F 0 "#FLG039" H 1100 1145 50  0001 C CNN
 F 1 "PWR_FLAG" H 1100 1230 50  0000 C CNN
 F 2 "" H 1100 1050 60  0000 C CNN
@@
 $EndComp
 $Comp
-L PWR_FLAG #FLG2
+L PWR_FLAG #FLG040
 U 1 1 56635DC4
 P 1650 1000
-F 0 "#FLG2" H 1650 1095 50  0001 C CNN
+F 0 "#FLG040" H 1650 1095 50  0001 C CNN
 F 1 "PWR_FLAG" H 1650 1180 50  0000 C CNN
 F 2 "" H 1650 1000 60  0000 C CNN
@@
 $EndComp
 $Comp
-L +BATT #PWR38
+L +BATT #PWR041
 U 1 1 5664A279
 P 2850 2150
-F 0 "#PWR38" H 2850 2000 50  0001 C CNN
+F 0 "#PWR041" H 2850 2000 50  0001 C CNN
 F 1 "+BATT" H 2850 2290 50  0000 C CNN
 F 2 "" H 2850 2150 60  0000 C CNN
@@
 F 0 "Q5" H 3575 2225 60  0000 C CNN
 F 1 "AO3401" H 3750 2125 60  0000 C CNN
-F 2 "SMD_Packages:SOT-323" H 2900 2290 60  0001 C CNN
+F 2 "CustomSmd:SOT23" H 2900 2290 60  0001 C CNN
 F 3 "" H 2900 2290 60  0000 C CNN
 	1    3350 2150
@@
 Enable5V
 $Comp
-L GND #PWR40
+L GND #PWR042
 U 1 1 5664A27D
 P 4500 2350
-F 0 "#PWR40" H 4500 2100 50  0001 C CNN
+F 0 "#PWR042" H 4500 2100 50  0001 C CNN
 F 1 "GND" H 4500 2200 50  0000 C CNN
 F 2 "" H 4500 2350 60  0000 C CNN
@@
 $EndComp
 $Comp
-L GND #PWR39
+L GND #PWR043
 U 1 1 5664A27F
 P 3850 2450
-F 0 "#PWR39" H 3850 2200 50  0001 C CNN
+F 0 "#PWR043" H 3850 2200 50  0001 C CNN
 F 1 "GND" H 3850 2300 50  0000 C CNN
 F 2 "" H 3850 2450 60  0000 C CNN
@@
 $EndComp
 $Comp
-L GND #PWR41
+L GND #PWR044
 U 1 1 5664A282
 P 5750 2350
-F 0 "#PWR41" H 5750 2100 50  0001 C CNN
+F 0 "#PWR044" H 5750 2100 50  0001 C CNN
 F 1 "GND" H 5750 2200 50  0000 C CNN
 F 2 "" H 5750 2350 60  0000 C CNN
@@
 Connection ~ 5750 2050
 $Comp
-L +5V #PWR42
+L +5V #PWR045
 U 1 1 5664A283
 P 6150 2050
-F 0 "#PWR42" H 6150 1900 50  0001 C CNN
+F 0 "#PWR045" H 6150 1900 50  0001 C CNN
 F 1 "+5V" H 6150 2190 50  0000 C CNN
 F 2 "" H 6150 2050 60  0000 C CNN
@@
 5V Supply
 $Comp
-L PWR_FLAG #FLG3
+L PWR_FLAG #FLG046
 U 1 1 5664A284
 P 3750 2000
-F 0 "#FLG3" H 3750 2095 50  0001 C CNN
+F 0 "#FLG046" H 3750 2095 50  0001 C CNN
 F 1 "PWR_FLAG" H 3750 2180 50  0000 C CNN
 F 2 "" H 3750 2000 60  0000 C CNN
@@
 	3750 2000 3750 2150
 $Comp
-L VCC #PWR37
+L VCC #PWR047
 U 1 1 5664A479
 P 1800 1000
-F 0 "#PWR37" H 1800 850 50  0001 C CNN
+F 0 "#PWR047" H 1800 850 50  0001 C CNN
 F 1 "VCC" H 1800 1150 50  0000 C CNN
 F 2 "" H 1800 1000 60  0000 C CNN

Commit message: Use 0603 resistors
Signed-off-by: Philip Luyckx <philip.luyckx@gmail.com>
Parts:
- R11: footprint Resistors_SMD:R_1206 -> Resistors_SMD:R_0603
Changed lines of the file:
@@
 F 0 "R11" V 3080 2450 50  0000 C CNN
 F 1 "47k" V 3000 2450 50  0000 C CNN
-F 2 "Resistors_SMD:R_1206" V 2930 2450 30  0001 C CNN
+F 2 "Resistors_SMD:R_0603" V 2930 2450 30  0001 C CNN
 F 3 "" H 3000 2450 30  0000 C CNN
 	1    3000 2450
