File: Supply.sch (KiCad schematic (older format))
At the start: 11 parts, among them P3 CONN_01X02, Q1 AO3401, U4 TPS79718, U5 EPL3015, U6 TPS61222

Commit message: Update connectors to custom ones
Signed-off-by: Philip Luyckx <philip.luyckx@gmail.com>
Parts:
- P3: footprint Socket_Strips:Socket_Strip_Straight_1x02 -> PinHeaders:Pin_Header_Straight_1x02_TH
Changed lines of the file:
@@
 F 0 "P3" H 1800 2250 50  0000 C CNN
 F 1 "CONN_01X02" V 1900 2100 50  0000 C CNN
-F 2 "Socket_Strips:Socket_Strip_Straight_1x02" H 1800 2100 60  0001 C CNN
+F 2 "PinHeaders:Pin_Header_Straight_1x02_TH" H 1800 2100 60  0001 C CNN
 F 3 "" H 1800 2100 60  0000 C CNN
 	1    1800 2100
@@
 $EndComp
 $Comp
-L +BATT #PWR40
+L +BATT #PWR038
 U 1 1 56631049
 P 1600 2050
-F 0 "#PWR40" H 1600 1900 50  0001 C CNN
+F 0 "#PWR038" H 1600 1900 50  0001 C CNN
 F 1 "+BATT" H 1600 2190 50  0000 C CNN
 F 2 "" H 1600 2050 60  0000 C CNN
@@
 $EndComp
 $Comp
-L GND #PWR41
+L GND #PWR039
 U 1 1 5663105F
 P 1600 2150
-F 0 "#PWR41" H 1600 1900 50  0001 C CNN
+F 0 "#PWR039" H 1600 1900 50  0001 C CNN
 F 1 "GND" H 1600 2000 50  0000 C CNN
 F 2 "" H 1600 2150 60  0000 C CNN
@@
 	1400 2400 1400 1800
 $Comp
-L +BATT #PWR39
+L +BATT #PWR040
 U 1 1 56635CFE
 P 1500 1000
-F 0 "#PWR39" H 1500 850 50  0001 C CNN
+F 0 "#PWR040" H 1500 850 50  0001 C CNN
 F 1 "+BATT" H 1500 1140 50  0000 C CNN
 F 2 "" H 1500 1000 60  0000 C CNN
@@
 $EndComp
 $Comp
-L GND #PWR38
+L GND #PWR041
 U 1 1 56635D42
 P 1100 1050
-F 0 "#PWR38" H 1100 800 50  0001 C CNN
+F 0 "#PWR041" H 1100 800 50  0001 C CNN
 F 1 "GND" H 1100 900 50  0000 C CNN
 F 2 "" H 1100 1050 60  0000 C CNN
@@
 $EndComp
 $Comp
-L PWR_FLAG #FLG1
+L PWR_FLAG #FLG042
 U 1 1 56635D80
 P 1100 1050
-F 0 "#FLG1" H 1100 1145 50  0001 C CNN
+F 0 "#FLG042" H 1100 1145 50  0001 C CNN
 F 1 "PWR_FLAG" H 1100 1230 50  0000 C CNN
 F 2 "" H 1100 1050 60  0000 C CNN
@@
 $EndComp
 $Comp
-L PWR_FLAG #FLG2
+L PWR_FLAG #FLG043
 U 1 1 56635DC4
 P 1650 1000
-F 0 "#FLG2" H 1650 1095 50  0001 C CNN
+F 0 "#FLG043" H 1650 1095 50  0001 C CNN
 F 1 "PWR_FLAG" H 1650 1180 50  0000 C CNN
 F 2 "" H 1650 1000 60  0000 C CNN
@@
 $EndComp
 $Comp
-L +BATT #PWR43
+L +BATT #PWR044
 U 1 1 5664A279
 P 2850 2150
-F 0 "#PWR43" H 2850 2000 50  0001 C CNN
+F 0 "#PWR044" H 2850 2000 50  0001 C CNN
 F 1 "+BATT" H 2850 2290 50  0000 C CNN
 F 2 "" H 2850 2150 60  0000 C CNN
@@
 Enable5V
 $Comp
-L GND #PWR49
+L GND #PWR045
 U 1 1 5664A27D
 P 4500 2350
-F 0 "#PWR49" H 4500 2100 50  0001 C CNN
+F 0 "#PWR045" H 4500 2100 50  0001 C CNN
 F 1 "GND" H 4500 2200 50  0000 C CNN
 F 2 "" H 4500 2350 60  0000 C CNN
@@
 $EndComp
 $Comp
-L GND #PWR47
+L GND #PWR046
 U 1 1 5664A27F
 P 3850 2450
-F 0 "#PWR47" H 3850 2200 50  0001 C CNN
+F 0 "#PWR046" H 3850 2200 50  0001 C CNN
 F 1 "GND" H 3850 2300 50  0000 C CNN
 F 2 "" H 3850 2450 60  0000 C CNN
@@
 $EndComp
 $Comp
-L GND #PWR50
+L GND #PWR047
 U 1 1 5664A282
 P 5750 2350
-F 0 "#PWR50" H 5750 2100 50  0001 C CNN
+F 0 "#PWR047" H 5750 2100 50  0001 C CNN
 F 1 "GND" H 5750 2200 50  0000 C CNN
 F 2 "" H 5750 2350 60  0000 C CNN
@@
 Connection ~ 5750 2050
 $Comp
-L +5V #PWR51
+L +5V #PWR048
 U 1 1 5664A283
 P 6150 2050
-F 0 "#PWR51" H 6150 1900 50  0001 C CNN
+F 0 "#PWR048" H 6150 1900 50  0001 C CNN
 F 1 "+5V" H 6150 2190 50  0000 C CNN
 F 2 "" H 6150 2050 60  0000 C CNN
@@
 5V Supply
 $Comp
-L PWR_FLAG #FLG3
+L PWR_FLAG #FLG049
 U 1 1 5664A284
 P 3750 2000
-F 0 "#FLG3" H 3750 2095 50  0001 C CNN
+F 0 "#FLG049" H 3750 2095 50  0001 C CNN
 F 1 "PWR_FLAG" H 3750 2180 50  0000 C CNN
 F 2 "" H 3750 2000 60  0000 C CNN
@@
 	3750 2000 3750 2150
 $Comp
-L VCC #PWR42
+L VCC #PWR050
 U 1 1 5664A479
 P 1800 1000
-F 0 "#PWR42" H 1800 850 50  0001 C CNN
+F 0 "#PWR050" H 1800 850 50  0001 C CNN
 F 1 "VCC" H 1800 1150 50  0000 C CNN
 F 2 "" H 1800 1000 60  0000 C CNN
@@
 $EndComp
 $Comp
-L +BATT #PWR45
+L +BATT #PWR051
 U 1 1 5752E781
 P 3500 3750
-F 0 "#PWR45" H 3500 3600 50  0001 C CNN
+F 0 "#PWR051" H 3500 3600 50  0001 C CNN
 F 1 "+BATT" H 3500 3890 50  0000 C CNN
 F 2 "" H 3500 3750 50  0000 C CNN
@@
 $EndComp
 $Comp
-L GND #PWR44
+L GND #PWR052
 U 1 1 5752E7D6
 P 3200 4300
-F 0 "#PWR44" H 3200 4050 50  0001 C CNN
+F 0 "#PWR052" H 3200 4050 50  0001 C CNN
 F 1 "GND" H 3200 4150 50  0000 C CNN
 F 2 "" H 3200 4300 50  0000 C CNN
@@
 $EndComp
 $Comp
-L GND #PWR48
+L GND #PWR053
 U 1 1 5752E81C
 P 4400 3850
-F 0 "#PWR48" H 4400 3600 50  0001 C CNN
+F 0 "#PWR053" H 4400 3600 50  0001 C CNN
 F 1 "GND" H 4400 3700 50  0000 C CNN
 F 2 "" H 4400 3850 50  0000 C CNN
@@
 1V8 Supply\n
 $Comp
-L +1V8 #PWR46
+L +1V8 #PWR054
 U 1 1 5753ACA5
 P 3500 3950
-F 0 "#PWR46" H 3500 3800 50  0001 C CNN
+F 0 "#PWR054" H 3500 3800 50  0001 C CNN
 F 1 "+1V8" H 3500 4090 50  0000 C CNN
 F 2 "" H 3500 3950 50  0000 C CNN
