File: Sensors.sch (KiCad schematic (older format))
At the start: 26 parts, among them Q4 Q_NMOS_GSD, U1 MCP60x4, U2 HTU21D, U3 PIR

Commit message: Add prices
Signed-off-by: Philip Luyckx <philip.luyckx@gmail.com>
Parts:
- C10, C8, C9, Q4: Price (none) -> 0.02
- R15, R16, R17, R20, R5: Price (none) -> 0.01
- U1: Price (none) -> 0.58
- U2: Price (none) -> 2.15
Connections:
- net VCC renamed +BATT
Changed lines of the file:
@@
 F 2 "Resistors_SMD:R_0603" V 2530 1900 30  0001 C CNN
 F 3 "" H 2600 1900 30  0000 C CNN
+F 4 "0.01" V 2600 1900 60  0001 C CNN "Price"
 	1    2600 1900
 	0    1    1    0
@@
 F 2 "CustomSmd:HTU21D_QFN" H 1950 3800 60  0001 C CNN
 F 3 "" H 1950 3800 60  0000 C CNN
+F 4 "2.15" H 1950 3800 60  0001 C CNN "Price"
 	1    1950 3800
 	1    0    0    -1
@@
 F 2 "Resistors_SMD:R_0805" H 1288 3850 50  0001 C CNN
 F 3 "" H 1250 4000 50  0000 C CNN
+F 4 "0.02" H 1250 4000 60  0001 C CNN "Price"
 	1    1250 4000
 	1    0    0    -1
@@
 F 2 "CustomSmd:SOIC-14" H 2650 1150 60  0001 C CNN
 F 3 "" H 2650 1150 60  0000 C CNN
+F 4 "0.58" H 2650 1150 60  0001 C CNN "Price"
 	3    2650 1150
 	1    0    0    -1
@@
 F 2 "CustomSmd:SOIC-14" H 7200 3750 60  0001 C CNN
 F 3 "" H 7200 3750 60  0000 C CNN
+F 4 "0.58" H 7200 3750 60  0001 C CNN "Price"
 	1    7200 3750
 	1    0    0    -1
@@
 F 2 "CustomSmd:SOIC-14" H 1900 5550 60  0001 C CNN
 F 3 "" H 1900 5550 60  0000 C CNN
+F 4 "0.58" H 1900 5550 60  0001 C CNN "Price"
 	5    1900 5550
 	1    0    0    -1
@@
 F 2 "Resistors_SMD:R_0805" H 1438 5600 50  0001 C CNN
 F 3 "" H 1400 5750 50  0000 C CNN
+F 4 "0.02" H 1400 5750 60  0001 C CNN "Price"
 	1    1400 5750
 	1    0    0    -1
@@
 F 2 "Resistors_SMD:R_0805" H 1188 5600 50  0001 C CNN
 F 3 "" H 1150 5750 50  0000 C CNN
+F 4 "0.02" H 1150 5750 60  0001 C CNN "Price"
 	1    1150 5750
 	1    0    0    -1
@@
 F 2 "Resistors_SMD:R_0603" V 8680 3700 50  0001 C CNN
 F 3 "" H 8750 3700 50  0000 C CNN
+F 4 "0.01" V 8750 3700 60  0001 C CNN "Price"
 	1    8750 3700
 	1    0    0    -1
@@
 F 2 "Resistors_SMD:R_0603" V 8680 4200 50  0001 C CNN
 F 3 "" H 8750 4200 50  0000 C CNN
+F 4 "0.01" V 8750 4200 60  0001 C CNN "Price"
 	1    8750 4200
 	1    0    0    -1
@@
 F 2 "Resistors_SMD:R_0603" V 9580 3650 50  0001 C CNN
 F 3 "" H 9650 3650 50  0000 C CNN
+F 4 "0.01" V 9650 3650 60  0001 C CNN "Price"
 	1    9650 3650
 	0    1    1    0
@@
 F 2 "CustomSmd:SOT23" H 10400 4150 50  0001 C CNN
 F 3 "" H 10200 4050 50  0000 C CNN
+F 4 "0.02" H 10200 4050 60  0001 C CNN "Price"
 	1    10200 4050
 	1    0    0    -1
@@
 F 2 "Resistors_SMD:R_0603" V 10230 3700 50  0001 C CNN
 F 3 "" H 10300 3700 50  0000 C CNN
+F 4 "0.01" V 10300 3700 60  0001 C CNN "Price"
 	1    10300 3700
 	1    0    0    -1
 $EndComp
 $Comp
-L VCC #PWR037
-U 1 1 58973B27
+L +BATT #PWR037
+U 1 1 58A791D4
 P 10300 3550
 F 0 "#PWR037" H 10300 3400 50  0001 C CNN
-F 1 "VCC" H 10300 3700 50  0000 C CNN
+F 1 "+BATT" H 10300 3690 50  0000 C CNN
 F 2 "" H 10300 3550 50  0000 C CNN
 F 3 "" H 10300 3550 50  0000 C CNN
